File: hardware/pcb/board/mainboard/mainboard.kicad_pcb (KiCad board)
At the start: 2 copper layers, 10 parts, among them J2 Conn_02x40_Odd_Even_MountingP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, J3 Conn_02x40_Odd_Even_MountingP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, J4 Conn_02x35_Odd_Even_MountingP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, J6 2908-05WB-MG, U2 STUSB4500QTR, U3 NEO-M8N, U4 LSM6DS3TR, U6 LIS2MDL, U7 BQ27441-G1, U9 TPS7A20_SOT-23

Commit message: USB PD AP33771C
Parts:
- added Q1: DMN3008SFG, Package_SON:Diodes_PowerDI3333-8, F.Cu at (192.6, 46.6)
- added Q3: DMN3008SFG, Package_SON:Diodes_PowerDI3333-8, F.Cu at (186.5, 46.6)
- added R1: 330, Resistor_SMD:R_0603_1608Metric_Pad0.98x0.95mm_HandSolder, F.Cu at (242.5, 92.3)
- added R10: 5mO, Resistor_SMD:R_0603_1608Metric_Pad0.98x0.95mm_HandSolder, F.Cu at (179.7, 46.3)
- added R11: 200, Resistor_SMD:R_0603_1608Metric_Pad0.98x0.95mm_HandSolder, F.Cu at (251.2, 92.3)
- added R12: 6.2k, Resistor_SMD:R_0603_1608Metric_Pad0.98x0.95mm_HandSolder, F.Cu at (251.2, 94.8)
- added R13: 100k, Resistor_SMD:R_0603_1608Metric_Pad0.98x0.95mm_HandSolder, F.Cu at (251.2, 97.3)
- added R2: 1.8M, Resistor_SMD:R_0603_1608Metric_Pad0.98x0.95mm_HandSolder, F.Cu at (242.5, 94.8)
- added R3: 10 mΩ, 1%, Resistor_SMD:R_0603_1608Metric_Pad0.98x0.95mm_HandSolder, F.Cu at (242.5, 97.3)
- added R4: 2.2k, Resistor_SMD:R_0603_1608Metric_Pad0.98x0.95mm_HandSolder, F.Cu at (242.5, 99.8)
- added R5: 10k, Resistor_SMD:R_0603_1608Metric_Pad0.98x0.95mm_HandSolder, F.Cu at (242.5, 102.3)
- added R6: 10k, Resistor_SMD:R_0603_1608Metric_Pad0.98x0.95mm_HandSolder, F.Cu at (246.8, 92.3)
- added R7: 5.1k, Resistor_SMD:R_0603_1608Metric_Pad0.98x0.95mm_HandSolder, F.Cu at (246.8, 94.8)
- added R8: 5.1k, Resistor_SMD:R_0603_1608Metric_Pad0.98x0.95mm_HandSolder, F.Cu at (246.8, 97.3)
- added R9: 1k, Resistor_SMD:R_0603_1608Metric_Pad0.98x0.95mm_HandSolder, F.Cu at (246.8, 99.8)

Commit message: PCB stackup
Parts:
- moved J2 52.6 mm to (125.2, 76.5)
- moved J3 52.6 mm to (146.8, 80.2)
- moved J4 52.6 mm to (132.4, 91.4)
Other:
- copper layers 2 -> 6
Changed lines of the file:
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@@
 	(generator_version "8.0")
 	(general
-		(thickness 1.6)
+		(thickness 1.635)
 		(legacy_teardrops no)
 	)
@@
 	(layers
 		(0 "F.Cu" signal)
+		(1 "In1.Cu" power "GND0")
+		(2 "In2.Cu" signal "HS Signal")
+		(3 "In3.Cu" power "PWR")
+		(4 "In4.Cu" power "GND1")
 		(31 "B.Cu" signal)
 		(32 "B.Adhes" user "B.Adhesive")
@@
 	)
 	(setup
+		(stackup
+			(layer "F.SilkS"
+				(type "Top Silk Screen")
+			)
+			(layer "F.Paste"
+				(type "Top Solder Paste")
+			)
+			(layer "F.Mask"
+				(type "Top Solder Mask")
+				(thickness 0.01)
+			)
+			(layer "F.Cu"
+				(type "copper")
+				(thickness 0.035)
+			)
+			(layer "dielectric 1"
+				(type "prepreg")
+				(thickness 0.23)
+				(material "FR4")
+				(epsilon_r 4.25)
+				(loss_tangent 0.02)
+			)
+			(layer "In1.Cu"
+				(type "copper")
+				(thickness 0.035)
+			)
+			(layer "dielectric 2"
+				(type "core")
+				(thickness 0.3)
+				(material "FR4")
+				(epsilon_r 4.5)
+				(loss_tangent 0.02)
+			)
+			(layer "In2.Cu"
+				(type "copper")
+				(thickness 0.035)
+			)
+			(layer "dielectric 3"
+				(type "prepreg")
+				(thickness 0.345)
+				(material "FR4")
+				(epsilon_r 4.25)
+				(loss_tangent 0.02)
+			)
+			(layer "In3.Cu"
+				(type "copper")
+				(thickness 0.035)
+			)
+			(layer "dielectric 4"
+				(type "core")
+				(thickness 0.3)
+				(material "FR4")
+				(epsilon_r 4.5)
+				(loss_tangent 0.02)
+			)
+			(layer "In4.Cu"
+				(type "copper")
+				(thickness 0.035)
+			)
+			(layer "dielectric 5"
+				(type "prepreg")
+				(thickness 0.23)
+				(material "FR4")
+				(epsilon_r 4.25)
+				(loss_tangent 0.02)
+			)
+			(layer "B.Cu"
+				(type "copper")
+				(thickness 0.035)
+			)
+			(layer "B.Mask"
+				(type "Bottom Solder Mask")
+				(thickness 0.01)
+			)
+			(layer "B.Paste"
+				(type "Bottom Solder Paste")
+			)
+			(layer "B.SilkS"
+				(type "Bottom Silk Screen")
+			)
+			(copper_finish "None")
+			(dielectric_constraints no)
+		)
 		(pad_to_mask_clearance 0)
 		(allow_soldermask_bridges_in_footprints no)
@@
 	(footprint "unsurv_offline_pcb_footprints:DF40_3.0_80"
 		(layer "F.Cu")
-		(at 78.5 52.3 -90)
+		(at 125.25 76.5 -90)
 		(property "Reference" "J2"
 			(at 8.83 -2.63 -90)
@@
 	(footprint "unsurv_offline_pcb_footprints:DF40_3.0_70"
 		(layer "F.Cu")
-		(at 85.69 67.17)
+		(at 132.44 91.37)
 		(property "Reference" "J4"
 			(at 7.21 -2.52 0)
@@
 	(footprint "unsurv_offline_pcb_footprints:DF40_3.0_80"
 		(layer "F.Cu")
-		(at 100 56.04 -90)
+		(at 146.75 80.24 -90)
 		(property "Reference" "J3"
 			(at 8.83 -2.63 -90)
@@
 		(tags "PowerDI 0.65")
 		(property "Reference" "Q3"
-			(at 0 -2.65 360)
+			(at 0 -2.65 0)
 			(layer "F.SilkS")
 			(effects
@@
 		)
 		(property "Value" "DMN3008SFG"
-			(at 0 2.65 360)
+			(at 0 2.65 0)
 			(layer "F.Fab")
 			(effects
@@
 		)
 		(fp_text user "${REFERENCE}"
-			(at 0 0 360)
+			(at 0 0 0)
 			(layer "F.Fab")
 			(effects
@@
 		(tags "PowerDI 0.65")
 		(property "Reference" "Q1"
-			(at 0 -2.65 360)
+			(at 0 -2.65 0)
 			(layer "F.SilkS")
 			(effects
@@
 		)
 		(property "Value" "DMN3008SFG"
-			(at 0 2.65 360)
+			(at 0 2.65 0)
 			(layer "F.Fab")
 			(effects
@@
 		)
 		(fp_text user "${REFERENCE}"
-			(at 0 0 360)
+			(at 0 0 0)
 			(layer "F.Fab")
 			(effects
@@
 	)
 	(gr_rect
-		(start 73.75 26.1)
-		(end 103.75 73.1)
+		(start 120.5 50.3)
+		(end 150.5 97.3)
 		(stroke
 			(width 0.1)

Commit message: updated battery holder for GNSS backup power
Parts:
- added BT1: Battery_Cell, Battery:BatteryHolder_Keystone_2998_1x6.8mm, F.Cu at (347.4, 60.3)
- added C1: 10 uF, Capacitor_SMD:C_0603_1608Metric, F.Cu at (312.1, 52.7)
- added C10: 100 nF, Capacitor_SMD:C_0603_1608Metric, F.Cu at (312.1, 75.3)
- added C11: 10 uF, Capacitor_SMD:C_0603_1608Metric, F.Cu at (312.1, 77.8)
- added C12: 10 uF, Capacitor_SMD:C_0603_1608Metric, F.Cu at (316.1, 52.7)
- added C13: 100 nF, Capacitor_SMD:C_0603_1608Metric, F.Cu at (316.1, 55.2)
- added C14: 100 nF, Capacitor_SMD:C_0603_1608Metric, F.Cu at (316.1, 57.8)
- added C15: 10 uF aluminium, Capacitor_SMD:C_0603_1608Metric, F.Cu at (316.1, 60.3)
- added C16: 100 nF, Capacitor_SMD:C_0603_1608Metric, F.Cu at (316.1, 62.8)
- added C17: 100 nF, Capacitor_SMD:C_0603_1608Metric, F.Cu at (316.1, 65.3)
- added C18: 220 nF, Capacitor_SMD:C_0603_1608Metric, F.Cu at (316.1, 67.8)
- added C19: 100 nF, Capacitor_SMD:C_0603_1608Metric, F.Cu at (316.1, 70.3)
- added C2: 1 uF, Capacitor_SMD:C_0603_1608Metric, F.Cu at (312.1, 55.2)
- added C20: 100 nF, Capacitor_SMD:C_0603_1608Metric, F.Cu at (316.1, 72.8)
- added C21: 22 uF, Capacitor_SMD:C_0603_1608Metric, F.Cu at (316.1, 75.3)
- added C22: 22 uF, Capacitor_SMD:C_0603_1608Metric, F.Cu at (316.1, 77.8)
- added C23: 22 uF, Capacitor_SMD:C_0603_1608Metric, F.Cu at (320.1, 52.7)
- added C24: 10 uF, Capacitor_SMD:C_0603_1608Metric, F.Cu at (320.1, 55.2)
- added C25: 1 uF, Capacitor_SMD:C_0603_1608Metric, F.Cu at (320.1, 57.8)
- added C26: 100 nF, Capacitor_SMD:C_0603_1608Metric, F.Cu at (320.1, 60.3)
- added C27: 100 nF, Capacitor_SMD:C_0603_1608Metric, F.Cu at (320.1, 62.8)
- added C28: 22 uF, Capacitor_SMD:C_0603_1608Metric, F.Cu at (320.1, 65.3)
- added C29: 1 uF, Capacitor_SMD:C_0603_1608Metric, F.Cu at (320.1, 67.8)
- added C3: 1 uF, Capacitor_SMD:C_0603_1608Metric, F.Cu at (312.1, 57.8)
- added C30: 1 uF, Capacitor_SMD:C_0603_1608Metric, F.Cu at (320.1, 70.3)
- added C31: 10 uF, Capacitor_SMD:C_0603_1608Metric, F.Cu at (320.1, 72.8)
- added C32: 100 nF, Capacitor_SMD:C_0603_1608Metric, F.Cu at (320.1, 75.3)
- added C33: 10 uF, Capacitor_SMD:C_0603_1608Metric, F.Cu at (320.1, 77.8)
- added C34: 100 nF, Capacitor_SMD:C_0603_1608Metric, F.Cu at (324.1, 52.7)
- added C35: 100 nF, Capacitor_SMD:C_0603_1608Metric, F.Cu at (324.1, 55.2)
- added C36: 100 nF, Capacitor_SMD:C_0603_1608Metric, F.Cu at (324.1, 57.8)
- added C37: 100 nF, Capacitor_SMD:C_0603_1608Metric, F.Cu at (324.1, 60.3)
- added C4: 47 nF, Capacitor_SMD:C_0603_1608Metric, F.Cu at (312.1, 60.3)
- added C5: 100 nF, Capacitor_SMD:C_0603_1608Metric, F.Cu at (312.1, 62.8)
- added C6: 1 uF, Capacitor_SMD:C_0603_1608Metric, F.Cu at (312.1, 65.3)
- added C7: 1 uF, Capacitor_SMD:C_0603_1608Metric, F.Cu at (312.1, 67.8)
- added C8: 0.47 uF, Capacitor_SMD:C_0603_1608Metric, F.Cu at (312.1, 70.3)
- added C9: 10 uF, Capacitor_SMD:C_0603_1608Metric, F.Cu at (312.1, 72.8)
- added D1: D, Diode_SMD:D_0603_1608Metric, F.Cu at (362.7, 52.8)
- added D2: LED, LED_SMD:LED_0603_1608Metric, F.Cu at (362.7, 55.4)
- added D3: LED, LED_SMD:LED_0603_1608Metric, F.Cu at (362.7, 58.0)
- added D4: LED, LED_SMD:LED_0603_1608Metric, F.Cu at (362.7, 60.5)
- added D5: LED_green, LED_SMD:LED_0603_1608Metric, F.Cu at (362.7, 63.1)
- added D6: LED, LED_SMD:LED_0603_1608Metric, F.Cu at (362.7, 65.7)
- added D7: LED, LED_SMD:LED_0603_1608Metric, F.Cu at (362.7, 68.3)
- added J1: Conn_Coaxial, Connector_Coaxial:SMA_Molex_73251-2200_Horizontal, F.Cu at (361.2, 92.9)
- added J10: USB_C_Receptacle, Connector_USB:USB_C_Receptacle_Amphenol_12401548E4-2A, F.Cu at (327.8, 85.5)
- added J2: BATTERY_Insta_360_Ace_Pro, Connector_PinHeader_2.00mm:PinHeader_1x04_P2.00mm_Vertical, F.Cu at (366.7, 53.5)
- added J6: USB_C_Receptacle, Connector_USB:USB_C_Receptacle_Amphenol_12401548E4-2A, F.Cu at (316.0, 85.5)
- added J7: Conn_01x30, Connector_FFC-FPC:Hirose_FH12-30S-0.5SH_1x30-1MP_P0.50mm_Horizontal, F.Cu at (345.2, 78.9)
- added J8: Conn_01x30, Connector_FFC-FPC:Hirose_FH12-30S-0.5SH_1x30-1MP_P0.50mm_Horizontal, F.Cu at (345.2, 87.9)
- added J9: Conn_01x30, Connector_FFC-FPC:Hirose_FH12-30S-0.5SH_1x30-1MP_P0.50mm_Horizontal, F.Cu at (345.2, 96.8)
- added JP1: Jumper_2_Small_Open, Jumper:SolderJumper-2_P1.3mm_Open_TrianglePad1.0x1.5mm, F.Cu at (318.2, 107.7)
- added L1: 1 uH, Inductor_SMD:L_0603_1608Metric, F.Cu at (324.1, 62.8)
- added L2: 1 uH, Inductor_SMD:L_0603_1608Metric, F.Cu at (324.1, 65.3)
- added Q1: BSS138, digikey-footprints:SOT-23-3, F.Cu at (367.0, 64.0)
- added R1: 1k, Resistor_SMD:R_0603_1608Metric, F.Cu at (324.1, 67.8)
- added R10: 10k, Resistor_SMD:R_0603_1608Metric, F.Cu at (328.1, 55.2)
- added R11: 10k, Resistor_SMD:R_0603_1608Metric, F.Cu at (328.1, 57.8)
- added R12: 2.2k, Resistor_SMD:R_0603_1608Metric, F.Cu at (328.1, 60.3)
- added R13: 5.23k, Resistor_SMD:R_0603_1608Metric, F.Cu at (328.1, 62.8)
- added R14: 30.1k, Resistor_SMD:R_0603_1608Metric, F.Cu at (328.1, 65.3)
- added R15: 3k, Resistor_SMD:R_0603_1608Metric, F.Cu at (328.1, 67.8)
- added R16: 316, Resistor_SMD:R_0603_1608Metric, F.Cu at (328.1, 70.3)
- added R17: 649, Resistor_SMD:R_0603_1608Metric, F.Cu at (328.1, 72.8)
- added R18: 5.1k, Resistor_SMD:R_0603_1608Metric, F.Cu at (328.1, 75.3)
- added R19: 5.1k, Resistor_SMD:R_0603_1608Metric, F.Cu at (328.1, 77.8)
- added R2: 0, Resistor_SMD:R_0603_1608Metric, F.Cu at (324.1, 70.3)
- added R25: 10k, Resistor_SMD:R_0603_1608Metric, F.Cu at (332.1, 52.7)
- added R28: 82k, Resistor_SMD:R_0603_1608Metric, F.Cu at (332.1, 55.2)
- added R29: 26k, Resistor_SMD:R_0603_1608Metric, F.Cu at (332.1, 57.8)
- added R3: 0, Resistor_SMD:R_0603_1608Metric, F.Cu at (324.1, 72.8)
- added R30: 10k, Resistor_SMD:R_0603_1608Metric, F.Cu at (332.1, 60.3)
- added R31: 10k, Resistor_SMD:R_0603_1608Metric, F.Cu at (332.1, 62.8)
- added R5: 0, Resistor_SMD:R_0603_1608Metric, F.Cu at (324.1, 75.3)
- added R6: 0, Resistor_SMD:R_0603_1608Metric, F.Cu at (324.1, 77.8)
- added R8: 2.2k, Resistor_SMD:R_0603_1608Metric, F.Cu at (328.1, 52.7)
- added TP1: TestPoint, TestPoint:TestPoint_Pad_D1.5mm, F.Cu at (311.8, 93.5)
- added TP10: TestPoint, TestPoint:TestPoint_Pad_D1.5mm, F.Cu at (318.9, 97.1)
- added TP11: TestPoint, TestPoint:TestPoint_Pad_D1.5mm, F.Cu at (318.9, 100.6)
- added TP12: TestPoint, TestPoint:TestPoint_Pad_D1.5mm, F.Cu at (318.9, 104.2)
- added TP13: TestPoint, TestPoint:TestPoint_Pad_D1.5mm, F.Cu at (322.5, 93.5)
- added TP14: TestPoint, TestPoint:TestPoint_Pad_D1.5mm, F.Cu at (322.5, 97.1)
- added TP15: TestPoint, TestPoint:TestPoint_Pad_D1.5mm, F.Cu at (322.5, 100.6)
- added TP16: TestPoint, TestPoint:TestPoint_Pad_D1.5mm, F.Cu at (322.5, 104.2)
- added TP17: TestPoint, TestPoint:TestPoint_Pad_D1.5mm, F.Cu at (326.0, 93.5)
- added TP18: TestPoint, TestPoint:TestPoint_Pad_D1.5mm, F.Cu at (326.0, 97.1)
- added TP19: TestPoint, TestPoint:TestPoint_Pad_D1.5mm, F.Cu at (326.0, 100.6)
- added TP2: TestPoint, TestPoint:TestPoint_Pad_D1.5mm, F.Cu at (311.8, 97.1)
- added TP20: TestPoint, TestPoint:TestPoint_Pad_D1.5mm, F.Cu at (326.0, 104.2)
- added TP21: TestPoint, TestPoint:TestPoint_Pad_D1.5mm, F.Cu at (329.6, 93.5)
- added TP22: TestPoint, TestPoint:TestPoint_Pad_D1.5mm, F.Cu at (329.6, 97.1)
- added TP23: TestPoint, TestPoint:TestPoint_Pad_D1.5mm, F.Cu at (329.6, 100.6)
- added TP24: TestPoint, TestPoint:TestPoint_Pad_D1.5mm, F.Cu at (329.6, 104.2)
- added TP3: TestPoint, TestPoint:TestPoint_Pad_D1.5mm, F.Cu at (311.8, 100.6)
- added TP4: TestPoint, TestPoint:TestPoint_Pad_D1.5mm, F.Cu at (311.8, 104.2)
- added TP5: TestPoint, TestPoint:TestPoint_Pad_D1.5mm, F.Cu at (315.4, 93.5)
- added TP6: TestPoint, TestPoint:TestPoint_Pad_D1.5mm, F.Cu at (315.4, 97.1)
- added TP7: TestPoint, TestPoint:TestPoint_Pad_D1.5mm, F.Cu at (315.4, 100.6)
- added TP8: TestPoint, TestPoint:TestPoint_Pad_D1.5mm, F.Cu at (315.4, 104.2)
- added TP9: TestPoint, TestPoint:TestPoint_Pad_D1.5mm, F.Cu at (318.9, 93.5)
- added U10: FT232RL, Package_SO:SSOP-28_5.3x10.2mm_P0.65mm, F.Cu at (361.6, 103.6)
- added U11: TPS7A20_SOT-23, Package_SON:Texas_X2SON-4_1x1mm_P0.65mm, F.Cu at (322.0, 107.2)
- added U12: AP33771C, unsurv_offline_pcb_footprints:DFN-14-1EP_3x3mm_P0.4mm_EP1.80x2.70mm, F.Cu at (363.7, 72.2)
- added U13: TXS0104E, Package_DFN_QFN:Texas_S-PVQFN-N14, F.Cu at (313.2, 107.7)
- added U4: BQ25606, Package_DFN_QFN:HVQFN-24-1EP_4x4mm_P0.5mm_EP2.6x2.6mm_ThermalVias, F.Cu at (346.7, 105.4)
- added U6: SN74LVC1T45DBVR, digikey-footprints:SOT-23-6, F.Cu at (336.5, 104.9)
- added U8: SN74LVC1T45DBVR, digikey-footprints:SOT-23-6, F.Cu at (341.2, 104.9)
- added U9: TPS61235P, unsurv_offline_pcb_footprints:cursed_TI-QFN9_TPS61235, F.Cu at (353.0, 105.4)
- R20: renamed from R10; footprint Resistor_SMD:R_0603_1608Metric_Pad0.98x0.95mm_HandSolder -> Resistor_SMD:R_0603_1608Metric
- R21: renamed from R13; footprint Resistor_SMD:R_0603_1608Metric_Pad0.98x0.95mm_HandSolder -> Resistor_SMD:R_0603_1608Metric
- R22: renamed from R11; footprint Resistor_SMD:R_0603_1608Metric_Pad0.98x0.95mm_HandSolder -> Resistor_SMD:R_0603_1608Metric
- R23: renamed from R12; footprint Resistor_SMD:R_0603_1608Metric_Pad0.98x0.95mm_HandSolder -> Resistor_SMD:R_0603_1608Metric
- R24: renamed from R7; footprint Resistor_SMD:R_0603_1608Metric_Pad0.98x0.95mm_HandSolder -> Resistor_SMD:R_0603_1608Metric
- R26: renamed from R8; footprint Resistor_SMD:R_0603_1608Metric_Pad0.98x0.95mm_HandSolder -> Resistor_SMD:R_0603_1608Metric
- R27: renamed from R9; footprint Resistor_SMD:R_0603_1608Metric_Pad0.98x0.95mm_HandSolder -> Resistor_SMD:R_0603_1608Metric
- R4: renamed from R3; footprint Resistor_SMD:R_0603_1608Metric_Pad0.98x0.95mm_HandSolder -> Resistor_SMD:R_0603_1608Metric
- R7: renamed from R1; footprint Resistor_SMD:R_0603_1608Metric_Pad0.98x0.95mm_HandSolder -> Resistor_SMD:R_0603_1608Metric
- R9: renamed from R2; footprint Resistor_SMD:R_0603_1608Metric_Pad0.98x0.95mm_HandSolder -> Resistor_SMD:R_0603_1608Metric
- moved Q2 131.7 mm to (318.2, 46.0)
- moved Q3 131.7 mm to (324.3, 46.0)
- moved R20 131.7 mm to (311.4, 45.8)
- moved J3 126.3 mm to (253.0, 53.9)
- moved J4 126.3 mm to (245.8, 39.0)
- moved J5 126.3 mm to (267.4, 42.7)
- renumbered J6 to J11, J4 to J3, J2 to J4, J3 to J5, Q3 to Q2, Q1 to Q3, U9 to U1, U4 to U2, U7 to U5, U6 to U7
Connections:
- net BATTERY_THERMISTOR renamed BATTERY_THERM
- J11 pad 1: unconnected-(J6-DAT2-Pad1) -> SD_DAT2
- J11 pad 2: unconnected-(J6-CD/DAT3-Pad2) -> SD_CS
- J11 pad 3: unconnected-(J6-CMD-Pad3) -> SD_CMD
- J11 pad 4: unconnected-(J6-VDD-Pad4) -> +3V3
- J11 pad 5: unconnected-(J6-CLK-Pad5) -> SD_CLK
- J11 pad 6: unconnected-(J6-VSS-Pad6) -> CE
- J11 pad 7: unconnected-(J6-DAT0-Pad7) -> DAT0
- J11 pad 8: unconnected-(J6-DAT1-Pad8) -> SD_DAT1
- J11 pad 9: unconnected-(J6-SHLD-Pad9) -> CE
- J3 pad 1: unconnected-(J4-Pin_1-Pad1) -> PCIE_PERST_N
- J3 pad 10: unconnected-(J4-Pin_10-Pad10) -> CE
- J3 pad 11: CSI1_DN2 -> DSI_CKN
- J3 pad 12: CSI1_CKN -> DSI_DN0
- J3 pad 13: CSI1_DP2 -> CE
- J3 pad 14: CSI1_CKP -> DSI_DP0
- J3 pad 15: unconnected-(J4-Pin_15-Pad15) -> DSI_DN2
- J3 pad 16: unconnected-(J4-Pin_16-Pad16) -> CE
- J3 pad 17: CSI1_DP0 -> DSI_DP2
- J3 pad 19: CSI1_DN0 -> CE
- J3 pad 2: unconnected-(J4-Pin_2-Pad2) -> PCIE_CLKREQ_N
- J3 pad 21: unconnected-(J4-Pin_21-Pad21) -> DSI_DN1
- J3 pad 22: unconnected-(J4-Pin_22-Pad22) -> CE
- J3 pad 23: H_GPIO_21 -> DSI_DP1
- J3 pad 24: unconnected-(J4-Pin_24-Pad24) -> H_GPIO_7
- J3 pad 25: H_GPIO_20 -> CE
- J3 pad 26: unconnected-(J4-Pin_26-Pad26) -> H_GPIO_15
- J3 pad 27: H_GPIO_19 -> H_GPIO_9
- J3 pad 28: H_GPIO_5 -> H_GPIO_25
- J3 pad 29: H_GPIO_18 -> H_UART_TXD_2
- J3 pad 3: unconnected-(J4-Pin_3-Pad3) -> BOOT MODE
- J3 pad 30: H_GPIO_2 -> CE
- J3 pad 31: unconnected-(J4-Pin_31-Pad31) -> H_UART_RXD_2
- J3 pad 32: H_GPIO_1 -> unconnected-(J3-Pin_32-Pad32)
- J3 pad 33: unconnected-(J4-Pin_33-Pad33) -> CE
- J3 pad 34: H_UART_RTS_2 -> unconnected-(J3-Pin_34-Pad34)
- J3 pad 35: unconnected-(J4-Pin_35-Pad35) -> PCIE_WAKE_N
- J3 pad 36: H_UART_CTS_2 -> CE
- J3 pad 37: unconnected-(J4-Pin_37-Pad37) -> H_UART_CTS_2
- J3 pad 38: PCIE_WAKE_N -> unconnected-(J3-Pin_38-Pad38)
- J3 pad 39: unconnected-(J4-Pin_39-Pad39) (its old number) -> H_UART_RTS_2
- J3 pad 4: unconnected-(J4-Pin_4-Pad4) -> DSI_DN3
- J3 pad 41: unconnected-(J4-Pin_41-Pad41) (its old number) -> H_GPIO_1
- J3 pad 42: H_UART_RXD_2 -> CE
- J3 pad 43: unconnected-(J4-Pin_43-Pad43) -> H_GPIO_2
- J3 pad 44: H_UART_TXD_2 -> H_GPIO_18
- J3 pad 45: H_GPIO_25 -> H_GPIO_5
- J3 pad 46: H_GPIO_9 -> H_GPIO_19
- J3 pad 47: H_GPIO_15 -> CE
- J3 pad 48: unconnected-(J4-Pin_48-Pad48) -> H_GPIO_20
- J3 pad 49: H_GPIO_7 -> unconnected-(J3-Pin_49-Pad49)
- J3 pad 5: CSI1_DN1 -> unconnected-(J3-Pin_5-Pad5)
- J3 pad 50: DSI_DP1 -> H_GPIO_21
- J3 pad 52: DSI_DN1 -> CE
- J3 pad 54: unconnected-(J4-Pin_54-Pad54) -> CSI1_DN0
- J3 pad 56: DSI_DP2 -> CSI1_DP0
- J3 pad 57: unconnected-(J4-Pin_57-Pad57) -> CE
- J3 pad 58: DSI_DN2 -> CE
- J3 pad 59: DSI_DP0 -> CSI1_CKP
- J3 pad 6: CSI1_DN3 -> DSI_DP3
- J3 pad 60: unconnected-(J4-Pin_60-Pad60) -> CSI1_DP2
- J3 pad 61: DSI_DN0 -> CSI1_CKN
- J3 pad 62: DSI_CKN -> CSI1_DN2
- J3 pad 63: unconnected-(J4-Pin_63-Pad63) -> CE
- J3 pad 64: DSI_CKP -> CE
- J3 pad 65: unconnected-(J4-Pin_65-Pad65) -> CSI1_DP3
- J3 pad 66: unconnected-(J4-Pin_66-Pad66) -> CSI1_DP1
- J3 pad 67: DSI_DP3 -> CSI1_DN3
- J3 pad 68: unconnected-(J4-Pin_68-Pad68) -> CSI1_DN1
- J3 pad 69: DSI_DN3 -> CE
- J3 pad 7: CSI1_DP1 -> CE
- J3 pad 70: BOOT MODE -> CE
- J3 pad 8: CSI1_DP3 -> CE
- J3 pad 9: unconnected-(J4-Pin_9-Pad9) -> DSI_CKP
- J4 pad 1: unconnected-(J2-Pin_1-Pad1) -> ETH_TRX3_N
- J4 pad 10: VDD_5V -> unconnected-(J4-Pin_10-Pad10)
- J4 pad 11: unconnected-(J2-Pin_11-Pad11) -> CE
- J4 pad 12: VDD_1V8 -> unconnected-(J4-Pin_12-Pad12)
- J4 pad 13: H_GPIO_11 -> ETH_TRX1_N
- J4 pad 14: VDD_1V8 -> CE
- J4 pad 15: unconnected-(J2-Pin_15-Pad15) -> ETH_TRX1_P
- J4 pad 16: VDD_1V8 -> unconnected-(J4-Pin_16-Pad16)
- J4 pad 17: unconnected-(J2-Pin_17-Pad17) -> CE
- J4 pad 18: VDD_1V8 -> unconnected-(J4-Pin_18-Pad18)
- J4 pad 19: unconnected-(J2-Pin_19-Pad19) -> ETH_TRX0_N
- J4 pad 2: VDD_5V -> CE
- J4 pad 20: unconnected-(J2-Pin_20-Pad20) -> CE
- J4 pad 21: H_BB_SPI_DQ3 -> ETH_TRX0_P
- J4 pad 22: unconnected-(J2-Pin_22-Pad22) -> USB_DP
- J4 pad 23: H_BB_SPI_DQ2 -> CE
- J4 pad 24: unconnected-(J2-Pin_24-Pad24) -> USB_DN
- J4 pad 25: unconnected-(J2-Pin_25-Pad25) -> LED_0/PHY_CFG_0
- J4 pad 26: unconnected-(J2-Pin_26-Pad26) -> CE
- J4 pad 27: unconnected-(J2-Pin_27-Pad27) -> LINK_ST/PHY_CRG1
- J4 pad 28: H_I2C1_SCL -> H_GPIO_10
- J4 pad 3: unconnected-(J2-Pin_3-Pad3) -> ETH_TRX3_P
- J4 pad 30: H_I2C1_SDA -> H_SPI_CSI
- J4 pad 31: unconnected-(J2-Pin_31-Pad31) -> H_I2C2_SCL
- J4 pad 32: H_BB_SPI_CLK -> H_BB_SPI_CS0
- J4 pad 33: unconnected-(J2-Pin_33-Pad33) -> H_I2C2_SDA
- J4 pad 34: H_BB_SPI_DQ1 -> H_SPI_RST
- J4 pad 35: unconnected-(J2-Pin_35-Pad35) -> CE
- J4 pad 36: H_BB_SPI_DQ0 -> CE
- J4 pad 37: unconnected-(J2-Pin_37-Pad37) -> H_GPIO_14
- J4 pad 38: USB_VBUSIN -> unconnected-(J4-Pin_38-Pad38)
- J4 pad 4: VDD_5V -> unconnected-(J4-Pin_4-Pad4)
- J4 pad 43: unconnected-(J2-Pin_43-Pad43) -> USB_VBUSIN
- J4 pad 44: H_GPIO_14 -> unconnected-(J4-Pin_44-Pad44)
- J4 pad 45: unconnected-(J2-Pin_45-Pad45) -> H_BB_SPI_DQ0
- J4 pad 47: H_SPI_RST -> H_BB_SPI_DQ1
- J4 pad 48: H_I2C2_SDA -> unconnected-(J4-Pin_48-Pad48)
- J4 pad 49: H_BB_SPI_CS0 -> H_BB_SPI_CLK
- J4 pad 5: unconnected-(J2-Pin_5-Pad5) -> CE
- J4 pad 50: H_I2C2_SCL -> unconnected-(J4-Pin_50-Pad50)
- J4 pad 51: H_SPI_CSI -> H_I2C1_SDA
- J4 pad 53: H_GPIO_10 -> H_I2C1_SCL
- J4 pad 54: LINK_ST/PHY_CRG1 -> unconnected-(J4-Pin_54-Pad54)
- J4 pad 56: LED_0/PHY_CFG_0 -> unconnected-(J4-Pin_56-Pad56)
- J4 pad 57: USB_DN -> unconnected-(J4-Pin_57-Pad57)
- J4 pad 58: unconnected-(J2-Pin_58-Pad58) -> H_BB_SPI_DQ2
- J4 pad 59: USB_DP -> unconnected-(J4-Pin_59-Pad59)
- J4 pad 6: VDD_5V -> unconnected-(J4-Pin_6-Pad6)
- J4 pad 60: ETH_TRX0_P -> H_BB_SPI_DQ3
- J4 pad 62: ETH_TRX0_N -> unconnected-(J4-Pin_62-Pad62)
- J4 pad 63: unconnected-(J2-Pin_63-Pad63) -> VDD_1V8
- J4 pad 65: unconnected-(J2-Pin_65-Pad65) -> VDD_1V8
- J4 pad 66: ETH_TRX1_P -> unconnected-(J4-Pin_66-Pad66)
- J4 pad 67: unconnected-(J2-Pin_67-Pad67) -> VDD_1V8
- J4 pad 68: ETH_TRX1_N -> H_GPIO_11
- J4 pad 69: unconnected-(J2-Pin_69-Pad69) -> VDD_1V8
- J4 pad 7: unconnected-(J2-Pin_7-Pad7) -> ETH_TRX2_N
- J4 pad 70: unconnected-(J2-Pin_70-Pad70) -> CE
- J4 pad 71: unconnected-(J2-Pin_71-Pad71) -> VDD_5V
- J4 pad 72: ETH_TRX2_P -> CE
- J4 pad 73: unconnected-(J2-Pin_73-Pad73) -> VDD_5V
- J4 pad 74: ETH_TRX2_N -> CE
- J4 pad 75: unconnected-(J2-Pin_75-Pad75) -> VDD_5V
- J4 pad 76: unconnected-(J2-Pin_76-Pad76) -> CE
- J4 pad 77: unconnected-(J2-Pin_77-Pad77) -> VDD_5V
- J4 pad 78: ETH_TRX3_P -> CE
- J4 pad 79: unconnected-(J2-Pin_79-Pad79) -> VDD_5V
- J4 pad 8: VDD_5V -> CE
- J4 pad 80: ETH_TRX3_N -> CE
- J4 pad 9: unconnected-(J2-Pin_9-Pad9) -> ETH_TRX2_P
- J5 pad 1: unconnected-(J3-Pin_1-Pad1) -> PCIE2_REF_CN_CLKP
- J5 pad 10: unconnected-(J3-Pin_10-Pad10) -> H_GPIO_27
- J5 pad 11: unconnected-(J3-Pin_11-Pad11) -> CE
- J5 pad 13: USB3_SS_TX_P -> H_GPIO_4
- J5 pad 14: unconnected-(J3-Pin_14-Pad14) -> GPIO1_6
- J5 pad 15: USB3_SS_TX_N -> GPIO1_7
- J5 pad 16: SYS_nRST -> unconnected-(J5-Pin_16-Pad16)
- J5 pad 17: unconnected-(J3-Pin_17-Pad17) -> CE
- J5 pad 18: unconnected-(J3-Pin_18-Pad18) (its old number) -> H_GPIO_26
- J5 pad 19: USB3_SS_RX_N -> PCIE_TX1_P
- J5 pad 2: CAM_XVS -> PCIE_RX0_N
- J5 pad 20: unconnected-(J3-Pin_20-Pad20) (its old number) -> H_GPIO_0
- J5 pad 21: USB3_SS_RX_P -> PCIE_TX1_N
- J5 pad 22: unconnected-(J3-Pin_22-Pad22) -> GPIO1_5
- J5 pad 23: unconnected-(J3-Pin_23-Pad23) -> CE
- J5 pad 24: H_I2S_SDI -> GPIO1_4
- J5 pad 25: H_PCIE_CLKREQ_N -> PCIE_RX1_P
- J5 pad 26: H_I2S_WS -> H_GPIO_24
- J5 pad 27: H_UART_RXD_1 -> PCIE_RX1_N
- J5 pad 28: H_I2S_SDO -> unconnected-(J5-Pin_28-Pad28)
- J5 pad 29: H_UART_TXD_1 -> CE
- J5 pad 3: unconnected-(J3-Pin_3-Pad3) -> PCIE2_REF_CN_CLKN
- J5 pad 30: H_I2S_SCK -> unconnected-(J5-Pin_30-Pad30)
- J5 pad 31: H_PCIE_WAKE_N -> PCIE_TX2_P
- J5 pad 33: unconnected-(J3-Pin_33-Pad33) -> PCIE_TX2_N
- J5 pad 35: H_PCIE_PERST_N -> CE
- J5 pad 37: H_UART_RXD_3 -> PCIE_RX2_P
- J5 pad 38: GPIO1_4 -> H_UART_TXD_3
- J5 pad 39: unconnected-(J3-Pin_39-Pad39) -> PCIE_RX2_N
- J5 pad 4: CAM_XHS -> PCIE_RX0_P
- J5 pad 41: unconnected-(J3-Pin_41-Pad41) -> CE
- J5 pad 42: PCIE_RX2_N -> CE
- J5 pad 43: H_UART_TXD_3 -> GPIO1_4
- J5 pad 44: PCIE_RX2_P -> H_UART_RXD_3
- J5 pad 46: unconnected-(J3-Pin_46-Pad46) -> H_PCIE_PERST_N
- J5 pad 48: PCIE_TX2_N -> CE
- J5 pad 5: unconnected-(J3-Pin_5-Pad5) -> CE
- J5 pad 50: PCIE_TX2_P -> H_PCIE_WAKE_N
- J5 pad 51: unconnected-(J3-Pin_51-Pad51) (its old number) -> H_I2S_SCK
- J5 pad 52: unconnected-(J3-Pin_52-Pad52) -> H_UART_TXD_1
- J5 pad 53: unconnected-(J3-Pin_53-Pad53) (its old number) -> H_I2S_SDO
- J5 pad 54: PCIE_RX1_N -> H_UART_RXD_1
- J5 pad 55: H_GPIO_24 -> H_I2S_WS
- J5 pad 56: PCIE_RX1_P -> H_PCIE_CLKREQ_N
- J5 pad 57: GPIO1_4 -> H_I2S_SDI
- J5 pad 58: unconnected-(J3-Pin_58-Pad58) -> CE
- J5 pad 59: GPIO1_5 -> unconnected-(J5-Pin_59-Pad59)
- J5 pad 6: unconnected-(J3-Pin_6-Pad6) -> CE
- J5 pad 60: PCIE_TX1_N -> USB3_SS_RX_P
- J5 pad 61: H_GPIO_0 -> CE
- J5 pad 62: PCIE_TX1_P -> USB3_SS_RX_N
- J5 pad 63: H_GPIO_26 -> unconnected-(J5-Pin_63-Pad63)
- J5 pad 64: unconnected-(J3-Pin_64-Pad64) -> CE
- J5 pad 65: unconnected-(J3-Pin_65-Pad65) -> SYS_nRST
- J5 pad 66: GPIO1_7 -> USB3_SS_TX_N
- J5 pad 67: GPIO1_6 -> unconnected-(J5-Pin_67-Pad67)
- J5 pad 68: H_GPIO_4 -> USB3_SS_TX_P
- J5 pad 7: unconnected-(J3-Pin_7-Pad7) -> PCIE_TX0_N
- J5 pad 71: H_GPIO_27 -> unconnected-(J5-Pin_71-Pad71)
- J5 pad 72: PCIE_TX0_P -> unconnected-(J5-Pin_72-Pad72)
- J5 pad 74: PCIE_TX0_N -> unconnected-(J5-Pin_74-Pad74)
- J5 pad 75: unconnected-(J3-Pin_75-Pad75) -> CE
- J5 pad 76: unconnected-(J3-Pin_76-Pad76) -> CE
- J5 pad 77: PCIE_RX0_P -> CAM_XHS
- J5 pad 78: PCIE2_REF_CN_CLKN -> unconnected-(J5-Pin_78-Pad78)
- J5 pad 79: PCIE_RX0_N -> CAM_XVS
- J5 pad 80: PCIE2_REF_CN_CLKP -> unconnected-(J5-Pin_80-Pad80)
- J5 pad 9: unconnected-(J3-Pin_9-Pad9) -> PCIE_TX0_P
- R24 pad 1: GND -> CE
- R26 pad 1: GND -> CE
- R4 pad 1: BATTERY_VOLTAGE -> B+
- R4 pad 2: Net-(U7-SRN) -> Net-(U5-BAT)
- U1 pad 2: GND -> CE
- U1 pad 5: +3V3 -> GNSS_3V3
- U2 pad 1: GND -> CE
- U2 pad 2: GND -> CE
- U2 pad 3: GND -> CE
- U2 pad 4: unconnected-(U4-INT1-Pad4) -> H_GPIO_26
- U2 pad 6: GND -> CE
- U2 pad 7: GND -> CE
- U2 pad 9: unconnected-(U4-INT2-Pad9) -> H_GPIO_24
- U3 pad 10: GND -> CE
- U3 pad 12: GND -> CE
- U3 pad 13: GND -> CE
- U3 pad 20: UART_RX1 -> UBLOX_TX_3V3
- U3 pad 21: UART_TX1 -> UBLOX_RX_3V3
- U3 pad 22: 3V3 -> V_BCKP
- U3 pad 23: 3V3 -> GNSS_3V3
- U3 pad 24: GND -> CE
- U3 pad 3: Net-(D1-A) -> PPS
- U3 pad 5: unconnected-(U3-USB_DM-Pad5) -> Net-(U3-USB_DM)
- U3 pad 6: unconnected-(U3-USB_DP-Pad6) -> Net-(U3-USB_DP)
- U3 pad 8: unconnected-(U3-~{RESET}-Pad8) -> Net-(U3-~{RESET})
- U5 pad 3: GND -> CE
- U5 pad 6: BATTERY_VOLTAGE -> Net-(U5-BAT)
- U5 pad 7: Net-(U7-SRN) -> Net-(U5-BAT)
- U5 pad 8: BATTERY_VOLTAGE -> B+
- U7 pad 6: GND -> CE
- U7 pad 7: unconnected-(U6-DRDY-Pad7) -> H_GPIO_27
- U7 pad 8: GND -> CE
- U7 pad 9: +3V3 -> GNSS_3V3

Commit message: rough grouping of ICs on PCB
Parts:
- removed the R4 at (242.5, 99.8)
- removed the R5 at (242.5, 102.3)
- removed the R6 at (246.8, 92.3)
- removed the U2 at (265.3, 79.3)
- J8: moved to B.Cu
- moved J7 242.0 mm to (112.0, 143.6), turned to 180 degrees
- moved J8 239.8 mm to (112.0, 143.6)
- moved J9 204.6 mm to (140.9, 109.0), turned to 180 degrees
- moved J1 201.2 mm to (161.2, 114.3), turned to -90 degrees
- moved J10 176.0 mm to (161.0, 141.5), turned to 90 degrees
- moved J2 153.6 mm to (214.2, 35.4)
- moved D2 148.5 mm to (217.1, 26.1)
- moved J5 145.6 mm to (151.4, 130.8)
- moved J3 145.6 mm to (137.1, 142.0)
- moved J4 145.6 mm to (129.9, 127.1)
- moved U7 132.3 mm to (370.4, 163.8)
- moved R24 120.1 mm to (344.5, 24.8)
- moved R26 120.1 mm to (344.5, 27.3)
- moved R22 119.1 mm to (341.6, 14.7), turned to 90 degrees
- moved Q1 118.6 mm to (253.3, 97.7)
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Connections:
- BT1 pad 2: CE -> GND
- C1 pad 1: CE -> GND
- C10 pad 2: CE -> GND
- C11 pad 2: CE -> GND
- C12 pad 2: CE -> GND
- C13 pad 2: CE -> GND
- C14 pad 2: CE -> GND
- C15 pad 1: CE -> GND
- C16 pad 2: CE -> GND
- C17 pad 1: CE -> GND
- C18 pad 2: CE -> GND
- C19 pad 2: CE -> GND
- C2 pad 2: CE -> GND
- C20 pad 2: CE -> GND
- C21 pad 2: CE -> GND
- C22 pad 2: CE -> GND
- C23 pad 2: CE -> GND
- C24 pad 2: CE -> GND
- C25 pad 2: CE -> GND
- C26 pad 1: CE -> GND
- C27 pad 1: CE -> GND
- C28 pad 2: CE -> GND
- C29 pad 2: CE -> GND
- C3 pad 2: CE -> GND
- C30 pad 2: CE -> GND
- C31 pad 2: CE -> GND
- C32 pad 2: CE -> GND
- C33 pad 2: CE -> GND
- C34 pad 2: CE -> GND
- C35 pad 2: CE -> GND
- C36 pad 2: CE -> GND
- C37 pad 2: CE -> GND
- C5 pad 1: CE -> GND
- C6 pad 2: CE -> GND
- C7 pad 1: CE -> GND
- C8 pad 1: CE -> GND
- C9 pad 2: CE -> GND
- D2 pad 1: CE -> GND
- D6 pad 1: CE -> GND
- D7 pad 1: CE -> GND
- J1 pad 2: CE -> GND
- J10 pad A1: CE -> GND
- J10 pad A12: CE -> GND
- J10 pad B1: CE -> GND
- J10 pad B12: CE -> GND
- J11 pad 6: CE -> GND
- J11 pad 9: CE -> GND
- J3 pad 10: CE -> GND
- J3 pad 13: CE -> GND
- J3 pad 16: CE -> GND
- J3 pad 19: CE -> GND
- J3 pad 22: CE -> GND
- J3 pad 25: CE -> GND
- J3 pad 30: CE -> GND
- J3 pad 33: CE -> GND
- J3 pad 36: CE -> GND
- J3 pad 42: CE -> GND
- J3 pad 47: CE -> GND
- J3 pad 52: CE -> GND
- J3 pad 57: CE -> GND
- J3 pad 58: CE -> GND
- J3 pad 63: CE -> GND
- J3 pad 64: CE -> GND
- J3 pad 69: CE -> GND
- J3 pad 7: CE -> GND
- J3 pad 70: CE -> GND
- J3 pad 8: CE -> GND
- J4 pad 11: CE -> GND
- J4 pad 14: CE -> GND
- J4 pad 17: CE -> GND
- J4 pad 2: CE -> GND
- J4 pad 20: CE -> GND
- J4 pad 23: CE -> GND
- J4 pad 26: CE -> GND
- J4 pad 35: CE -> GND
- J4 pad 36: CE -> GND
- J4 pad 5: CE -> GND
- J4 pad 70: CE -> GND
- J4 pad 72: CE -> GND
- J4 pad 74: CE -> GND
- J4 pad 76: CE -> GND
- J4 pad 78: CE -> GND
- J4 pad 8: CE -> GND
- J4 pad 80: CE -> GND
- J5 pad 11: CE -> GND
- J5 pad 17: CE -> GND
- J5 pad 23: CE -> GND
- J5 pad 29: CE -> GND
- J5 pad 35: CE -> GND
- J5 pad 41: CE -> GND
- J5 pad 42: CE -> GND
- J5 pad 48: CE -> GND
- J5 pad 5: CE -> GND
- J5 pad 58: CE -> GND
- J5 pad 6: CE -> GND
- J5 pad 61: CE -> GND
- J5 pad 64: CE -> GND
- J5 pad 75: CE -> GND
- J5 pad 76: CE -> GND
- J6 pad A1: CE -> GND
- J6 pad A12: CE -> GND
- J6 pad B1: CE -> GND
- J6 pad B12: CE -> GND
- J7 pad 15: CE -> GND
- J7 pad 18: CE -> GND
- J7 pad 21: CE -> GND
- J7 pad 24: CE -> GND
- J7 pad 27: CE -> GND
- J7 pad 30: CE -> GND
- J7 pad 4: CE -> GND
- J7 pad 5: CE -> GND
- J8 pad 15: CE -> GND
- J8 pad 18: CE -> GND
- J8 pad 21: CE -> GND
- J8 pad 24: CE -> GND
- J8 pad 27: CE -> GND
- J8 pad 30: CE -> GND
- J8 pad 4: CE -> GND
- J8 pad 5: CE -> GND
- J9 pad 5: CE -> GND
- Q1 pad 2: CE -> GND
- R11 pad 2: CE -> GND
- R14 pad 2: CE -> GND
- R16 pad 2: CE -> GND
- R17 pad 2: CE -> GND
- R18 pad 1: CE -> GND
- R19 pad 1: CE -> GND
- R24 pad 1: CE -> GND
- R26 pad 1: CE -> GND
- R28 pad 2: CE -> GND
- R29 pad 2: CE -> GND
- TP17 pad 1: CE -> GND
- U1 pad 2: CE -> GND
- U10 pad 18: CE -> GND
- U10 pad 21: CE -> GND
- U10 pad 25: CE -> GND
- U10 pad 7: CE -> GND
- U11 pad 2: CE -> GND
- U12 pad 15: CE -> GND
- U12 pad 5: CE -> GND
- U13 pad 7: CE -> GND
- U2 pad 1: CE -> GND
- U2 pad 2: CE -> GND
- U2 pad 3: CE -> GND
- U2 pad 6: CE -> GND
- U2 pad 7: CE -> GND
- U3 pad 10: CE -> GND
- U3 pad 12: CE -> GND
- U3 pad 13: CE -> GND
- U3 pad 24: CE -> GND
- U4 pad 17: CE -> GND
- U4 pad 18: CE -> GND
- U4 pad 6: CE -> GND
- U4 pad 9: CE -> GND
- U5 pad 3: CE -> GND
- U6 pad 2: CE -> GND
- U7 pad 6: CE -> GND
- U7 pad 8: CE -> GND
- U8 pad 2: CE -> GND
- U8 pad 5: CE -> GND
- U9 pad 1: CE -> GND
- U9 pad 4: CE -> GND
- U9 pad 5: CE -> GND
- U9 pad 8: CE -> GND
Other:
- board outline added: 65 x 50 mm
- board text added: "GNSS antenna"
